File: KiCad/Mainboard/Z-FIGHTER_Mainboard.sch (KiCad schematic (older format))
At the start: 40 parts, among them IC1 Z80SIO, J1 DB9_Male_MountingHoles, J2 DB9_Male_MountingHoles, J3 USB_B, J4 Conn_02x13_Odd_Even, J5 Conn_Parallel_User, J6 Conn_PATA, SW1 SW_Push, SW2 SW_DIP_x03, U1 AS6C4008-55PCN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

Commit message: Annotated Mainboard schematic
Connections:
- net PATA38: now reaches J6.38 (Pin_38), RN3.2 (R1)
- net PATA34: now reaches J6.34 (Pin_34), RN3.3 (R2)
- net PATA29: now reaches J6.29 (Pin_29), RN3.4 (R3)
Other:
- note added: "512K ROM"
- note added: "Accessory board PPI"
- note added: "Accessory board header"
- note added: "CompactFlash adapter header"
- note added: "DIP-3 for manual ROM paging"
- note added: "Decoupling capacitors\nUSB 2.0 standard specifies max of 10uF between Vbus and GND"
- note added: "Optional clock oscillator for SIO Ch.B"
- note added: "Power connector"
- note added: "RAM"
- note added: "ROM disable flip-flop\nfor CP/M and #RESET inverter\nfor 8255 PPI"
- note added: "RS-232 level shifters"
- note added: "SIO/O Ch.A"
- note added: "SIO/O Ch.B"
- note added: "SPLD address decoder"
- note added: "Supervisory circuit"
- note added: "System/SIO clock oscillator"
- note added: "User PPI"
- note added: "User parallel port"
- note added: "Z80 CPU"
- note added: "Z80 SIO/0 serial I/O peripheral"
- note removed: "USB 2.0 standard specifies max of 10uF between Vbus and GND"
- moved on the sheet: C1, C10, C11, C12, C13, C3, C4, C5, C6, C7, C8, C9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

Commit message: Cleaned up mainboard schema
Parts:
- IC1: symbol Z-FIGHTER_Mainboard:Z80SIO -> Z-FIGHTER_Mainboard-rescue:Z80SIO-Z-FIGHTER_Mainboard-Z-FIGHTER_Mainboard-rescue-Z-FIGHTER_Mainboard-rescue-Z-FIGHTER_M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
- U10: symbol Z-FIGHTER_Mainboard:DS1233 -> Z-FIGHTER_Mainboard-rescue:DS1233-Z-FIGHTER_Mainboard-Z-FIGHTER_Mainboard-rescue-Z-FIGHTER_Mainboard-rescue-Z-FIGHTER_M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
- U5, U6: symbol Z-FIGHTER_Mainboard:MAX203 -> Z-FIGHTER_Mainboard-rescue:MAX203-Z-FIGHTER_Mainboard-Z-FIGHTER_Mainboard-rescue-Z-FIGHTER_Mainboard-rescue-Z-FIGHTER_M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
- U7: symbol Z-FIGHTER_Mainboard:ATF22V10C -> Z-FIGHTER_Mainboard-rescue:ATF22V10C-Z-FIGHTER_Mainboard-Z-FIGHTER_Mainboard-rescue-Z-FIGHTER_Mainboard-rescue-Z-FIGHTE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
Other:
- note added: "JP2&JP3 1-1: CTS signal is honored on SIO Ch.A/B\nJP2&JP3 2-3: CTS signal is ignored on SIO Ch.A/B"
- note added: "ROM disable flip-flop for CP/M\nand #RESET inverter for 8255 PPI\n"
- note added: "Z80 Microprocessor"
- note removed: "JP2/JP3 1-1: CTS signal is honored on SIO Ch.A/B\nJP2/JP3 2-3: CTS signal is ignored on SIO Ch.A/B"
- note removed: "ROM disable flip-flop\nfor CP/M and #RESET inverter\nfor 8255 PPI"
- note removed: "Z80 CPU"
- moved on the sheet: C1, C10, C11, C12, C13, C2, C3, C4, C5, C6, C7, C8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

Commit message: Initial submit
Parts:
- added J7: Conn_02x03_Odd_Even, Connector_IDC:IDC-Header_2x03_P2.54mm_Horizontal, symbol Connector_Generic:Conn_02x03_Odd_Even
- added JP4, JP5: Jumper_2_Open, Connector_PinHeader_2.54mm:PinHeader_1x02_P2.54mm_Vertical, symbol Jumper:Jumper_2_Open
- added R2: 4.7KΩ, Resistor_THT:R_Axial_DIN0207_L6.3mm_D2.5mm_P7.62mm_Horizontal, symbol Device:R
- IC1: symbol Z-FIGHTER_Mainboard-rescue:Z80SIO-Z-FIGHTER_Mainboard-Z-FIGHTER_Mainboard-rescue-Z-FIGHTER_Mainboard-rescue-Z-FIGHTER_Mainboard-rescue -> Z-FIGHTER_Mainboard-rescue:Z80SIO-Z-FIGHTER_Mainboard-Z-FIGHTER_Mainboard-rescue-Z-FIGHTER_Mainboard-rescue-Z-FIGHTER_Mainboard-rescue-Z-FIGHTER_Mainboard-rescue
- U10: symbol Z-FIGHTER_Mainboard-rescue:DS1233-Z-FIGHTER_Mainboard-Z-FIGHTER_Mainboard-rescue-Z-FIGHTER_Mainboard-rescue-Z-FIGHTER_Mainboard-rescue -> Z-FIGHTER_Mainboard-rescue:DS1233-Z-FIGHTER_Mainboard-Z-FIGHTER_Mainboard-rescue-Z-FIGHTER_Mainboard-rescue-Z-FIGHTER_Mainboard-rescue-Z-FIGHTER_Mainboard-rescue
- U5, U6: symbol Z-FIGHTER_Mainboard-rescue:MAX203-Z-FIGHTER_Mainboard-Z-FIGHTER_Mainboard-rescue-Z-FIGHTER_Mainboard-rescue-Z-FIGHTER_Mainboard-rescue -> Z-FIGHTER_Mainboard-rescue:MAX203-Z-FIGHTER_Mainboard-Z-FIGHTER_Mainboard-rescue-Z-FIGHTER_Mainboard-rescue-Z-FIGHTER_Mainboard-rescue-Z-FIGHTER_Mainboard-rescue
- U7: symbol Z-FIGHTER_Mainboard-rescue:ATF22V10C-Z-FIGHTER_Mainboard-Z-FIGHTER_Mainboard-rescue-Z-FIGHTER_Mainboard-rescue-Z-FIGHTER_Mainboard-rescue -> Z-FIGHTER_Mainboard-rescue:ATF22V10C-Z-FIGHTER_Mainboard-Z-FIGHTER_Mainboard-rescue-Z-FIGHTER_Mainboard-rescue-Z-FIGHTER_Mainboard-rescue-Z-FIGHTER_Mainboard-rescue
Connections:
- net #INT: now also J7.3 (Pin_3)
- net CLOCK1: now also J7.5 (Pin_5)
- net CLOCK2: now also J7.6 (Pin_6)
- net GND: now also J7.1 (Pin_1)
- net VCC: now also J7.2 (Pin_2), JP4.2 (B), JP5.2 (B), R2.1; no longer U2.17 (~NMI~)
- net at J1.9: now also JP4.1 (A)
- net at J2.9: now also JP5.1 (A)
- new net #NMI: J7.4 (Pin_4), R2.2, U2.17 (~NMI~)
- no-connect marks 39 -> 37
Other:
- note added: "CPU control lines & external SIO Ch.B clock pin"
- moved on the sheet: C2, RN2, SW1, SW2, U10
