File: KiCad/AccessoryBoard/Z-FIGHTER_Accessory_Board.kicad_pcb (KiCad board)
At the start: 2 copper layers, 100 x 75 mm, 24 parts, among them J7 ST7920 Graphic LCD, J9 Conn_02x13_Odd_Even, Q1 BC337, Q2 BC337, SW1 Up (A0), SW2 Down (A1), SW3 Left (A2), SW4 Right (A3), SW5 A (A4), SW6 B (A5)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

Commit message: Accessory board rev. 1b
Adjusted accessory board LCD connector pins to be 7.62mm (2.54mm*3) apart from pins on LCD board for easier bridging
Parts:
- moved J7 4.38 mm to (116.5, 58.6)
Routing:
- net GND: track 23.5 -> 29.5 mm
- net PB7S: track 76.2 -> 80.6 mm
- net PB5S: track 76.2 -> 80.6 mm
- net PB4S: track 76.2 -> 80.6 mm
- net BLK: track 3.34 -> 7.72 mm
- net PC1S: track 75.1 -> 79.5 mm
- net PC0S: track 72.2 -> 76.6 mm
- net PB6S: track 76.2 -> 80.6 mm
- net PB3S: track 72.6 -> 77.0 mm
- net PB1S: track 83.5 -> 87.9 mm
- net PB0S: track 94.8 -> 99.2 mm
- net PB2S: track 80.8 -> 85.2 mm
- net PC2S: track 77.7 -> 82.0 mm
Other:
- board text added: "Accessory Board Rev. 1b"
- board text removed: "Accessory Board Rev. 1a"

Commit message: Gerber settings
Other:
- rule pad_to_mask_clearance: 0.051 -> 0
Changed lines of the file:
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@@
     (pad_size 6.4 6.4)
     (pad_drill 3.200001)
-    (pad_to_mask_clearance 0.051)
-    (solder_mask_min_width 0.25)
+    (pad_to_mask_clearance 0)
     (aux_axis_origin 0 0)
     (grid_origin 116.5 51)
@@
     (pcbplotparams
       (layerselection 0x010fc_ffffffff)
-      (usegerberextensions false)
+      (usegerberextensions true)
       (usegerberattributes false)
       (usegerberadvancedattributes false)
@@
       (outputformat 1)
       (mirror false)
-      (drillshape 1)
+      (drillshape 0)
       (scaleselection 1)
-      (outputdirectory ""))
+      (outputdirectory "C:/Users/nhull/Desktop/"))
   )
   (net 0 "")

Commit message: Added drawing of LCD module
Parts:
- J7: footprint Connector_PinSocket_2.54mm:PinSocket_1x20_P2.54mm_Horizontal -> Connector_PinSocket_2.54mm:PinSocket_1x20_P2.54mm_Vertical
- moved J9 53.2 mm to (137.3, 164.1)
- moved BZ1 53.2 mm to (139.3, 101.0)
- moved D2 53.2 mm to (145.8, 108.9)
- moved G*** 53.2 mm to (146.6, 158.1)
- moved J7 53.2 mm to (81.5, 98.6)
- moved Mount1 53.2 mm to (70.0, 101.0)
- moved Mount2 53.2 mm to (158.0, 101.0)
- moved Mount3 53.2 mm to (70.0, 164.0)
- moved Mount4 53.2 mm to (158.0, 164.0)
- moved Q1 53.2 mm to (81.5, 106.3)
- moved Q2 53.2 mm to (129.8, 106.3)
- moved RB1 53.2 mm to (86.6, 108.9)
- moved RB2 53.2 mm to (138.2, 113.4)
- moved REF** 53.2 mm to (74.5, 153.1)
- moved RN4 53.2 mm to (127.1, 160.3)
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Other:
- board text added: "LCD Module"
