File: KiCad/Audio_Loader/Audio_Loader.kicad_pcb (KiCad board)
At the start: 2 copper layers, 55.9 x 38.1 mm, 22 parts, among them J1 USB PWR, J2 DE-9 Female, J3 TS Jack, Q1 BC547, U1 LM741, U2 LM393, U3 MAX202

Commit message: Update Audio_Loader.kicad_pcb
Parts:
- J1: value USB PWR -> USB +5V

Commit message: Update Audio_Loader.kicad_pcb
Parts:
- J1: value USB +5V -> ◄USB Power
Routing:
- net PIN_9: track 31.3 -> 40.2 mm
- net VCC: track 7.62 -> 0.00 mm
Other:
- board text added: "ZF Audio Loader @tangent3D 2021 Rev. 0b"
- board text removed: "ZF Audio Loader @tangent3D 2021 Rev. 0a"
