File: hardware/peripherals/baud_generator/kicad/Baud_Generator.kicad_pcb (KiCad board)
At the start: 2 copper layers, 16.5 x 41 mm, 6 parts, among them J1 Conn_02x03_Odd_Even, J2 Conn_02x07_Odd_Even, U1 4024, X1 2.4576 MHz

Commit message: Changed connector footprint from 6 to 8 pins
Parts:
- J1: value Conn_02x03_Odd_Even -> Conn_02x04_Odd_Even
- moved J1 0.13 mm to (113.6, 59.0), turned to 0 degrees
Routing:
- net GND: track 70.0 -> 73.0 mm
- net VCC: track 31.9 -> 33.4 mm
- net CLOCK2: track 40.6 -> 39.8 mm
Other:
- outline, holes or cut-outs redrawn
