File: hardware/peripherals/baud_generator/kicad/Baud_Generator.sch (KiCad schematic (older format))
At the start: 6 parts, among them J1 Conn_02x03_Odd_Even, J2 Conn_02x07_Odd_Even, U1 4024, X1 2.4576 MHz

Commit message: Changed connector footprint from 6 to 8 pins
Parts:
- J1: value Conn_02x03_Odd_Even -> Conn_02x04_Odd_Even; symbol Connector_Generic:Conn_02x03_Odd_Even -> Connector_Generic:Conn_02x04_Odd_Even
Connections:
- no-connect marks 4 -> 6
Changed lines of the file:
@@
 	1    0    0    -1
 $EndComp
-NoConn ~ 3550 1350
+NoConn ~ 4050 1350
 $Comp
-L Connector_Generic:Conn_02x03_Odd_Even J1
+L Connector_Generic:Conn_02x04_Odd_Even J1
 U 1 1 61973F40
-P 3750 1350
-F 0 "J1" H 3800 1667 50  0000 C CNN
-F 1 "Conn_02x03_Odd_Even" H 3800 1576 50  0001 C CNN
-F 2 "Baud_Generator:ZF_CPU_Control_Header" H 3750 1350 50  0001 C CNN
-F 3 "~" H 3750 1350 50  0001 C CNN
-	1    3750 1350
-	1    0    0    -1
+P 3850 1350
+F 0 "J1" H 3900 1667 50  0000 C CNN
+F 1 "Conn_02x04_Odd_Even" H 3900 1576 50  0001 C CNN
+F 2 "Baud_Generator:ZF_CPU_Control_Header" H 3850 1350 50  0001 C CNN
+F 3 "~" H 3850 1350 50  0001 C CNN
+	1    3850 1350
+	-1   0    0    1
 $EndComp
 Wire Wire Line
@@
 L power:VCC #PWR0106
 U 1 1 6197994A
-P 4050 1250
-F 0 "#PWR0106" H 4050 1100 50  0001 C CNN
-F 1 "VCC" V 4065 1377 50  0000 L CNN
-F 2 "" H 4050 1250 50  0001 C CNN
-F 3 "" H 4050 1250 50  0001 C CNN
-	1    4050 1250
-	0    1    1    0
+P 3550 1450
+F 0 "#PWR0106" H 3550 1300 50  0001 C CNN
+F 1 "VCC" V 3565 1577 50  0000 L CNN
+F 2 "" H 3550 1450 50  0001 C CNN
+F 3 "" H 3550 1450 50  0001 C CNN
+	1    3550 1450
+	0    -1   -1   0
 $EndComp
-Text GLabel 3550 1450 0    50   Input ~ 0
+Text GLabel 4050 1250 2    50   Input ~ 0
 CLOCK2
 $Comp
 L power:GND #PWR0107
 U 1 1 6197CD0A
-P 3550 1250
-F 0 "#PWR0107" H 3550 1000 50  0001 C CNN
-F 1 "GND" H 3555 1077 50  0000 C CNN
-F 2 "" H 3550 1250 50  0001 C CNN
-F 3 "" H 3550 1250 50  0001 C CNN
-	1    3550 1250
-	0    1    1    0
+P 4050 1450
+F 0 "#PWR0107" H 4050 1200 50  0001 C CNN
+F 1 "GND" H 4055 1277 50  0000 C CNN
+F 2 "" H 4050 1450 50  0001 C CNN
+F 3 "" H 4050 1450 50  0001 C CNN
+	1    4050 1450
+	0    -1   -1   0
 $EndComp
-NoConn ~ 4050 1350
-NoConn ~ 4050 1450
+NoConn ~ 3550 1350
+NoConn ~ 3550 1250
+NoConn ~ 3550 1150
+NoConn ~ 4050 1150
 $EndSCHEMATC
