File: hardware/peripherals/usb_serial_power_module/KiCad/usb_serial_power_module.kicad_sch (KiCad schematic)
At the start: 23 parts, among them J1 USB_B_Mini, J2 DE-9, U1 CY7C65213-28PVXI, U2 TPS2061CDBVT, U3 MAX202

Commit message: Change digi-key link to female DE-9
Parts:
- J2: Digi-Key https://www.digikey.com/en/products/detail/assmann-wsw-components/A-DS-09-A-KG-T2S/1241804 -> https://www.digikey.com/en/products/detail/assmann-wsw-components/A-DF-09-A-KG-T2S/1241800
Changed lines of the file:
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@@
       (effects (font (size 1.27 1.27)) hide)
     )
-    (property "Digi-Key" "https://www.digikey.com/en/products/detail/assmann-wsw-components/A-DS-09-A-KG-T2S/1241804" (id 4) (at 58.42 134.62 90)
+    (property "Digi-Key" "https://www.digikey.com/en/products/detail/assmann-wsw-components/A-DF-09-A-KG-T2S/1241800" (id 4) (at 58.42 134.62 90)
       (effects (font (size 1.27 1.27)) hide)
     )
