File: hardware/peripherals/usb_serial_power_module/KiCad/usb_serial_power_module.kicad_pcb (KiCad board)
At the start: 2 copper layers, 40 x 31 mm, 24 parts, among them J1 USB_B_Mini, J2 SIO Ch. B (RS-232), U1 CY7C65213-28PVXI, U2 TPS2061CDBVT, U3 MAX202

Commit message: Routing
Routing:
- net GND: track 62.4 -> 60.9 mm
- net Net-(C6-Pad2): track 5.03 -> 4.25 mm
- net #RXLED: track 12.8 -> 12.0 mm
- net Net-(C7-Pad1): track 4.56 -> 3.94 mm
- net #TXLED: track 6.16 -> 5.57 mm
Other:
- board text added: "Z-FIGHTER USB Serial Adapter w/ Remote Pin 9 +5V Rev. 1"
- board text removed: "Z-FIGHTER USB Serial Adapter w/ Remote Pin 9 +5V Rev. 0"

Commit message: USB serial/power module
Parts:
- moved C1 78.3 mm to (20.6, 12.6)
- moved C10 78.3 mm to (14.7, 25.9)
- moved C2 78.3 mm to (20.6, 9.38)
- moved C3 78.3 mm to (20.6, 6.20)
- moved C4 78.3 mm to (15.8, 5.97)
- moved C5 78.3 mm to (27.0, 19.5)
- moved C6 78.3 mm to (36.5, 15.7)
- moved C7 78.3 mm to (14.7, 20.8)
- moved C8 78.3 mm to (20.6, 15.7)
- moved C9 78.3 mm to (15.8, 15.7)
- moved D1 78.3 mm to (27.0, 27.2)
- moved D2 78.3 mm to (20.6, 3.02)
- moved D3 78.3 mm to (36.5, 3.02)
- moved D4 78.3 mm to (36.5, 6.20)
- moved G*** 78.3 mm to (28.5, 15.5)
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